File: PCB/smartwatch.kicad_pcb (KiCad board)
At the start: 2 copper layers, 34.2 x 34.2 mm, 5 parts, among them J1 Conn_01x04_Pin, U1 STM32L432KBUx, U2 LSM6DS3, U3 W25Q128JVPIQ, U4 TP4056

Commit message: Added gyroscope
Parts:
- added REF**: C_01005_0402Metric, Capacitor_SMD:C_01005_0402Metric, F.Cu at (152.1, 91.4)
- moved U2 1.63 mm to (150.1, 96.5)
Changed lines of the file:
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@@
   )
   (footprint "Package_LGA:LGA-14_3x2.5mm_P0.5mm_LayoutBorder3x4y" (layer "F.Cu")
-    (at 151.13 95.25)
+    (at 150.114 96.52)
     (descr "LGA, 14 Pin (https://www.st.com/resource/en/datasheet/lsm6ds3tr-c.pdf), generated with kicad-footprint-generator ipc_noLead_generator.py")
     (tags "LGA NoLead")
@@
       (offset (xyz 0 0 0))
       (scale (xyz 1 1 1))
+      (rotate (xyz 0 0 0))
+    )
+  )
+  (footprint "Capacitor_SMD:C_01005_0402Metric" (layer "F.Cu")
+    (at 152.146 91.44)
+    (descr "Capacitor SMD 01005 (0402 Metric), square (rectangular) end terminal, IPC_7351 nominal, (Body size source: http://www.vishay.com/docs/20056/crcw01005e3.pdf), generated with kicad-footprint-generator")
+    (tags "capacitor")
+    (attr smd)
+    (fp_text reference "REF**" (at 0 -1) (layer "F.SilkS")
+        (effects (font (size 1 1) (thickness 0.15)))
+    )
+    (fp_text value "C_01005_0402Metric" (at 0 1) (layer "F.Fab")
+        (effects (font (size 1 1) (thickness 0.15)))
+    )
+    (fp_text user "${REFERENCE}" (at 0 -0.62) (layer "F.Fab")
+        (effects (font (size 0.25 0.25) (thickness 0.04)))
+    )
+    (fp_line (start -0.6 -0.3) (end 0.6 -0.3)
+      (stroke (width 0.05) (type solid)) (layer "F.CrtYd"))
+    (fp_line (start -0.6 0.3) (end -0.6 -0.3)
+      (stroke (width 0.05) (type solid)) (layer "F.CrtYd"))
+    (fp_line (start 0.6 -0.3) (end 0.6 0.3)
+      (stroke (width 0.05) (type solid)) (layer "F.CrtYd"))
+    (fp_line (start 0.6 0.3) (end -0.6 0.3)
+      (stroke (width 0.05) (type solid)) (layer "F.CrtYd"))
+    (fp_line (start -0.2 -0.1) (end 0.2 -0.1)
+      (stroke (width 0.1) (type solid)) (layer "F.Fab"))
+    (fp_line (start -0.2 0.1) (end -0.2 -0.1)
+      (stroke (width 0.1) (type solid)) (layer "F.Fab"))
+    (fp_line (start 0.2 -0.1) (end 0.2 0.1)
+      (stroke (width 0.1) (type solid)) (layer "F.Fab"))
+    (fp_line (start 0.2 0.1) (end -0.2 0.1)
+      (stroke (width 0.1) (type solid)) (layer "F.Fab"))
+    (pad "" smd roundrect (at -0.275 0) (size 0.27 0.27) (layers "F.Paste") (roundrect_rratio 0.25))
+    (pad "" smd roundrect (at 0.275 0) (size 0.27 0.27) (layers "F.Paste") (roundrect_rratio 0.25))
+    (pad "1" smd roundrect (at -0.25 0) (size 0.4 0.3) (layers "F.Cu" "F.Mask") (roundrect_rratio 0.25))
+    (pad "2" smd roundrect (at 0.25 0) (size 0.4 0.3) (layers "F.Cu" "F.Mask") (roundrect_rratio 0.25))
+    (model "${KICAD6_3DMODEL_DIR}/Capacitor_SMD.3dshapes/C_01005_0402Metric.wrl"
+      (offset (xyz 0 0 0))
+      (scale (xyz 1 1 1))

Commit message: new staffz
Parts:
- removed REF**: C_01005_0402Metric, Capacitor_SMD:C_01005_0402Metric
- added C1: 4.7uf, Capacitor_SMD:C_0603_1608Metric, F.Cu at (153.7, 84.3)
- added C10: 100nf, Capacitor_SMD:C_0603_1608Metric, F.Cu at (153.7, 89.7)
- added C11: 4.7uf, Capacitor_SMD:C_0603_1608Metric, F.Cu at (162.3, 82.8)
- added C12: 4.7uf, Capacitor_SMD:C_0603_1608Metric, F.Cu at (164.1, 82.8)
- added C13: 4.7uf, Capacitor_SMD:C_0603_1608Metric, F.Cu at (156.5, 90.7)
- added C2: 100nf, Capacitor_SMD:C_0603_1608Metric, F.Cu at (153.7, 91.4)
- added C3: 100nf, Capacitor_SMD:C_0603_1608Metric, F.Cu at (149.4, 90.7)
- added C4: 100nf, Capacitor_SMD:C_0603_1608Metric, F.Cu at (151.1, 90.7)
- added C5: 100nf, Capacitor_SMD:C_0603_1608Metric, F.Cu at (149.1, 97.5)
- added C6: 9pf, Capacitor_SMD:C_0603_1608Metric, F.Cu at (149.1, 95.7)
- added C7: 9pf, Capacitor_SMD:C_0603_1608Metric, F.Cu at (149.1, 93.2)
- added C8: 100nf, Capacitor_SMD:C_0603_1608Metric, F.Cu at (153.7, 87.9)
- added C9: 100nf, Capacitor_SMD:C_0603_1608Metric, F.Cu at (153.7, 86.1)
- added U5: LT1761-3.3, Package_TO_SOT_SMD:TSOT-23-5, F.Cu at (159.3, 90.0)
- added X2: 20Mhz, Crystal:Crystal_SMD_3225-4Pin_3.2x2.5mm, F.Cu at (165.1, 92.2)
- added Y2: LSE 32khz, Crystal:Crystal_SMD_3215-2Pin_3.2x1.5mm, F.Cu at (152.1, 94.5)
- J1: value Conn_01x04_Pin -> Serial wire/Charging
- moved J1 21.0 mm to (153.4, 79.2), turned to 90 degrees
- moved U4 13.7 mm to (159.2, 84.7), turned to 90 degrees
- moved U2 5.34 mm to (149.9, 101.9)
- moved U3 3.04 mm to (155.4, 102.7), turned to 90 degrees
- moved U1 2.34 mm to (157.0, 95.5)
Connections:
- J1 pad 3: unconnected-(J1-Pin_3-Pad3) -> VIN
- J1 pad 4: unconnected-(J1-Pin_4-Pad4) -> GND
- U1 pad 1: unconnected-(U1-VDD-Pad1) -> VDD
- U1 pad 12: unconnected-(U1-PA6-Pad12) -> SPI1_MISO
- U1 pad 13: unconnected-(U1-PA7-Pad13) -> SPI1_MOSI
- U1 pad 16: Net-(U1-VSS-Pad16) -> GND
- U1 pad 17: unconnected-(U1-VDD-Pad17) -> VDD
- U1 pad 2: unconnected-(U1-PC14-Pad2) -> OSC32_IN
- U1 pad 3: unconnected-(U1-PC15-Pad3) -> OSC32_OUT
- U1 pad 32: Net-(U1-VSS-Pad16) -> GND
- U1 pad 33: Net-(U1-VSS-Pad16) -> GND
- U1 pad 4: unconnected-(U1-NRST-Pad4) -> Net-(U1-NRST)
- U1 pad 5: unconnected-(U1-VDDA-Pad5) -> VDD
- U1 pad 6: unconnected-(U1-PA0-Pad6) -> CLKIN
- U1 pad 7: unconnected-(U1-PA1-Pad7) -> SPI1_SCK
- U2 pad 1: unconnected-(U2-SDO/SA0-Pad1) -> SPI1_MISO
- U2 pad 12: unconnected-(U2-CS-Pad12) -> GYRO_CS
- U2 pad 13: unconnected-(U2-SCL-Pad13) -> SPI1_SCK
- U2 pad 14: unconnected-(U2-SDA-Pad14) -> SPI1_MISO
- U2 pad 2: unconnected-(U2-SDX-Pad2) -> GND
- U2 pad 3: unconnected-(U2-SCX-Pad3) -> GND
- U2 pad 4: unconnected-(U2-INT1-Pad4) -> GYRO_INT1
- U2 pad 5: unconnected-(U2-VDDIO-Pad5) -> VDD
- U2 pad 6: Net-(U2-GND-Pad6) -> GND
- U2 pad 7: Net-(U2-GND-Pad6) -> GND
- U2 pad 8: unconnected-(U2-VDD-Pad8) -> VDD
- U2 pad 9: unconnected-(U2-INT2-Pad9) -> GYRO_INT2
- U3 pad 1: unconnected-(U3-/CS-Pad1) -> FLASH_CS
- U3 pad 2: unconnected-(U3-DO_(IO1)-Pad2) -> SPI1_MISO
- U3 pad 3: unconnected-(U3-/WP_(IO2)-Pad3) -> VDD
- U3 pad 4: (no net) -> GND
- U3 pad 5: unconnected-(U3-DI_(IO0)-Pad5) -> SPI1_MOSI
- U3 pad 6: unconnected-(U3-CLK-Pad6) -> SPI1_SCK
- U3 pad 7: unconnected-(U3-/HOLD_or_/RESET_(IO3)-Pad7) -> HR_FLASH
- U3 pad 8: unconnected-(U3-VCC-Pad8) -> VDD
- U3 pad 9: unconnected-(U3-Pad9) -> GND
- U4 pad 1: unconnected-(U4-TEMP-Pad1) -> GND
- U4 pad 2: unconnected-(U4-PROG-Pad2) -> Net-(U4-PROG)
- U4 pad 3: unconnected-(U4-GND-Pad3) -> GND
- U4 pad 4: unconnected-(U4-VCC-Pad4) -> VIN
- U4 pad 5: unconnected-(U4-BAT-Pad5) -> BAT
- U4 pad 7: unconnected-(U4-~{CHRG}-Pad7) -> CHARGE
- U4 pad 8: unconnected-(U4-CE-Pad8) -> VIN
- U4 pad 9: unconnected-(U4-PP-Pad9) -> GND
Routing:
- net GND: track 0.00 -> 89.1 mm, vias 0 -> 20
- net VDD: track 0.00 -> 70.5 mm, vias 0 -> 17
- net BAT: track 0.00 -> 13.9 mm
- net SPI1_MISO: track 0.00 -> 8.21 mm, vias 0 -> 2
- net Net-(U1-NRST): track 0.00 -> 6.51 mm
- net OSC32_IN: track 0.00 -> 5.08 mm
- net OSC32_OUT: track 0.00 -> 5.07 mm
- net SPI1_SCK: track 0.00 -> 4.70 mm
- net VIN: track 0.00 -> 3.12 mm
- net SPI1_MOSI: track 0.00 -> 2.09 mm
- net Net-(U5-BYP): track 0.00 -> 1.96 mm
- added copper zone on In1.Cu, net GND
- added copper zone on In2.Cu, net VDD
Other:
- copper layers 2 -> 4

Commit message: files?
Parts:
- added REF**: PCB Edge, Connector_FFC-FPC:TE_1-1734839-5_1x15-1MP_P0.5mm_Horizontal, F.Cu at (171.8, 93.5)
- moved C9 18.9 mm to (149.1, 104.5), turned to 90 degrees
- moved C8 18.9 mm to (146.4, 105.3)
- moved C1 16.9 mm to (162.8, 98.6), turned to 90 degrees
- moved C10 16.8 mm to (154.3, 106.5), turned to 90 degrees
- moved X2 15.3 mm to (151.6, 99.4)
- moved C4 12.7 mm to (161.0, 98.6)
- moved C13 7.25 mm to (162.6, 86.8)
- moved U5 7.19 mm to (165.4, 86.2)
- moved C3 6.77 mm to (152.2, 96.8), turned to 0 degrees
- moved C5 5.94 mm to (143.2, 97.1), turned to -90 degrees
- moved U3 4.03 mm to (158.5, 105.2), turned to 0 degrees
- moved U2 3.54 mm to (146.5, 103.0)
- moved C12 2.38 mm to (166.3, 82.1), turned to -90 degrees
- moved C11 2.29 mm to (164.5, 82.0), turned to 90 degrees
- moved C2 1.65 mm to (155.3, 91.4)
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Connections:
- J1 pad 1: unconnected-(J1-Pin_1-Pad1) -> SWCLK
- J1 pad 2: unconnected-(J1-Pin_2-Pad2) -> SWDIO
- U1 pad 11: unconnected-(U1-PA5-Pad11) -> FLASH_SCK
- U1 pad 12: SPI1_MISO -> FLASH_MISO
- U1 pad 13: SPI1_MOSI -> FLASH_MOSI
- U1 pad 18: unconnected-(U1-PA8-Pad18) -> FLASH_CS
- U1 pad 24: unconnected-(U1-PA14-Pad24) -> SWCLK
- U1 pad 25: unconnected-(U1-PA15-Pad25) -> SWDIO
- U1 pad 26: unconnected-(U1-PB3-Pad26) -> GYRO_SCK
- U1 pad 27: unconnected-(U1-PB4-Pad27) -> GYRO_MISO
- U1 pad 28: unconnected-(U1-PB5-Pad28) -> GYRO_MOSI
- U1 pad 29: unconnected-(U1-PB6-Pad29) -> GYRO_CS
- U1 pad 7: SPI1_SCK -> BAT
- U2 pad 1: SPI1_MISO -> GYRO_MISO
- U2 pad 13: SPI1_SCK -> GYRO_SCK
- U2 pad 14: SPI1_MISO -> GYRO_MOSI
- U3 pad 2: SPI1_MISO -> FLASH_MISO
- U3 pad 6: SPI1_SCK -> FLASH_SCK
Routing:
- net GND: track 89.1 -> 0.00 mm, vias 20 -> 0
- net VDD: track 70.5 -> 0.00 mm, vias 17 -> 0
- net BAT: track 13.9 -> 0.00 mm
- net SPI1_MISO: track 8.21 -> 0.00 mm, vias 2 -> 0
- net Net-(U1-NRST): track 6.51 -> 0.00 mm
- net OSC32_IN: track 5.08 -> 0.00 mm
- net OSC32_OUT: track 5.07 -> 0.00 mm
- net SPI1_SCK: track 4.70 -> 0.00 mm
- net VIN: track 3.12 -> 0.00 mm
- net SPI1_MOSI: track 2.09 -> 0.00 mm
- net Net-(U5-BYP): track 1.96 -> 0.00 mm
Other:
- board size 34.2 x 34.2 mm -> 36 x 36 mm

Commit message: tighter pcb
Parts:
- moved J1 31.6 mm to (161.3, 109.1), turned to -90 degrees
- moved C11 22.7 mm to (152.2, 101.1), turned to -90 degrees
- moved C12 22.7 mm to (154.0, 101.1), turned to 90 degrees
- moved U5 22.4 mm to (153.2, 105.0)
- moved C13 22.3 mm to (150.2, 105.3)
- moved C8 22.3 mm to (163.4, 90.8)
- moved C9 22.3 mm to (166.1, 90.0)
- moved U2 22.3 mm to (163.5, 88.5)
- moved U4 21.0 mm to (158.4, 105.2), turned to 180 degrees
- moved C10 9.81 mm to (162.1, 100.5), turned to -90 degrees
- moved C5 8.09 mm to (148.1, 90.8)
- moved U3 6.47 mm to (158.1, 98.8), turned to -90 degrees
- moved C1 3.92 mm to (163.9, 94.8)
- moved C2 3.92 mm to (156.4, 87.7)
- moved C3 3.92 mm to (153.3, 93.1)
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
Commit message: All but routing done
Parts:
- removed the REF** at (171.8, 93.5)
- added ?: , , F.Cu at (168.4, 83.8)
- added C14: 100nf, Capacitor_SMD:C_0603_1608Metric, F.Cu at (162.6, 101.6)
- added C15: 100nf, Capacitor_SMD:C_0603_1608Metric, F.Cu at (166.8, 89.0)
- added C16: 100nf, Capacitor_SMD:C_0603_1608Metric, F.Cu at (160.4, 104.2)
- added D1: D, Diode_SMD:D_0201_0603Metric, F.Cu at (158.4, 85.4)
- added D2: D, Diode_SMD:D_0201_0603Metric, F.Cu at (159.2, 105.1)
- added J2: Battery input, Connector_PinHeader_2.54mm:PinHeader_1x02_P2.54mm_Vertical, F.Cu at (165.4, 104.7)
- added J3: Conn_01x15, Connector_FFC-FPC:TE_1-1734839-5_1x15-1MP_P0.5mm_Horizontal, F.Cu at (172.3, 93.8)
- added J4: Conn_01x03, Connector_FFC-FPC:TE_0-1734839-5_1x05-1MP_P0.5mm_Horizontal, F.Cu at (163.3, 86.8)
- added J5: USB_B_Micro, Connector_USB:USB_Micro-B_Amphenol_10118194_Horizontal, F.Cu at (157.6, 79.4)
- added R1: 15k, Resistor_SMD:R_0805_2012Metric, F.Cu at (162.4, 104.2)
- added R10: 4.7k, Resistor_SMD:R_0805_2012Metric, F.Cu at (161.4, 97.4)
- added R2: 1R, Resistor_SMD:R_0805_2012Metric, F.Cu at (146.4, 100.0)
- added R3: 10k, Resistor_SMD:R_0805_2012Metric, F.Cu at (166.0, 101.8)
- added R4: 1R, Resistor_SMD:R_0805_2012Metric, F.Cu at (150.8, 96.6)
- added R5: 4.7k, Resistor_SMD:R_0805_2012Metric, F.Cu at (146.6, 84.2)
- added R6: 4.7k, Resistor_SMD:R_0805_2012Metric, F.Cu at (154.0, 83.6)
- added R7: [Jumper], Resistor_SMD:R_0805_2012Metric, F.Cu at (147.0, 97.2)
- added R8: [Jumper], Resistor_SMD:R_0805_2012Metric, F.Cu at (142.4, 99.0)
- added R9: 4.7k, Resistor_SMD:R_0805_2012Metric, F.Cu at (144.8, 97.2)
- added REF**: MountingHole_2.2mm_M2_DIN965_Pad, MountingHole:MountingHole_2.2mm_M2_DIN965_Pad, F.Cu at (145.9, 103.6)
- added SW1: SW_SPDT, MyButtons:MSK12CO2, F.Cu at (149.2, 92.9)
- added U6: INA3221, Package_DFN_QFN:Texas_RGV0016A_VQFN-16-1EP_4x4mm_P0.65mm_EP2.1x2.1mm, F.Cu at (165.2, 98.0)
- added U8: USBLC6-2SC6, Package_TO_SOT_SMD:SOT-23-6, F.Cu at (164.5, 80.2)
- J1: footprint Connector_PinHeader_2.54mm:PinHeader_1x04_P2.54mm_Horizontal -> Connector_PinHeader_2.54mm:PinHeader_1x04_P2.54mm_Vertical
- moved C5 18.7 mm to (166.8, 92.2)
- moved C9 16.4 mm to (150.4, 85.2), turned to 180 degrees
- moved U2 15.2 mm to (150.4, 80.8)
- moved C8 14.9 mm to (150.4, 83.6)
- moved C10 4.30 mm to (159.4, 97.2)
- moved U1 3.31 mm to (155.5, 89.7)
- moved C2 3.31 mm to (153.8, 85.7)
- moved C3 3.31 mm to (150.7, 91.1)
- moved C6 3.31 mm to (148.2, 89.5)
- moved X2 3.31 mm to (150.1, 93.7)
- moved Y2 3.31 mm to (151.0, 88.2)
- moved C7 3.31 mm to (148.2, 87.0)
- moved C4 3.26 mm to (160.2, 92.2), turned to 180 degrees
- moved U4 3.07 mm to (155.6, 104.0)
- moved U3 2.98 mm to (155.5, 97.3)
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Connections:
- C5 pad 1: Net-(U1-NRST) -> GND
- C5 pad 2: GND -> VDD
- J1 pad 1: SWCLK -> Net-(J1-Pin_1)
- J1 pad 2: SWDIO -> Net-(J1-Pin_2)
- J1 pad 3: VIN -> Net-(D2-A)
- U1 pad 10: unconnected-(U1-PA4-Pad10) -> HEARTBEAT_AOUT
- U1 pad 11: FLASH_SCK -> CHARGE
- U1 pad 12: FLASH_MISO -> LEDA
- U1 pad 13: FLASH_MOSI -> GYRO_INT1
- U1 pad 14: unconnected-(U1-PB0-Pad14) -> QUADSPI_IO1
- U1 pad 15: unconnected-(U1-PB1-Pad15) -> QUADSPI_IO0
- U1 pad 18: FLASH_CS -> LCD_RS
- U1 pad 19: unconnected-(U1-PA9-Pad19) -> I2C1_SCL
- U1 pad 20: unconnected-(U1-PA10-Pad20) -> I2C1_SDA
- U1 pad 21: unconnected-(U1-PA11-Pad21) -> USB_DM
- U1 pad 22: unconnected-(U1-PA12-Pad22) -> USB_DP
- U1 pad 23: unconnected-(U1-PA13-Pad23) -> SWDIO
- U1 pad 25: SWDIO -> LCD_NSS
- U1 pad 26: GYRO_SCK -> LCD_SCK
- U1 pad 27: GYRO_MISO -> GYRO_INT2
- U1 pad 28: GYRO_MOSI -> LCD_MOSI
- U1 pad 29: GYRO_CS -> TP_INT
- U1 pad 30: unconnected-(U1-PB7-Pad30) -> TP_RST
- U1 pad 31: unconnected-(U1-PH3-Pad31) -> Net-(U1-PH3)
- U1 pad 4: Net-(U1-NRST) -> unconnected-(U1-NRST-Pad4)
- U1 pad 8: unconnected-(U1-PA2-Pad8) -> QUADSPI_NCS
- U1 pad 9: unconnected-(U1-PA3-Pad9) -> QUADSPI_CLK
- U2 pad 1: GYRO_MISO -> GND
- U2 pad 12: GYRO_CS -> VDD
- U2 pad 13: GYRO_SCK -> I2C1_SCL
- U2 pad 14: GYRO_MOSI -> I2C1_SDA
- U3 pad 1: FLASH_CS -> QUADSPI_NCS
- U3 pad 2: FLASH_MISO -> QUADSPI_IO1
- U3 pad 5: SPI1_MOSI -> QUADSPI_IO0
- U3 pad 6: FLASH_SCK -> QUADSPI_CLK
- U3 pad 7: HR_FLASH -> VDD
- U5 pad 1: BAT -> BATSHUNTH
- U5 pad 3: BAT -> BATSHUNTH
Other:
- board text added: "1"
- board text added: "15"
- board text added: "5"
- board text added: "5v"
- board text added: "BAT+"
- board text added: "GND"
- board text added: "SWCLK"
- board text added: "SWDIO"

Commit message: pcb done
Parts:
- removed R8: [Jumper], Resistor_SMD:R_0805_2012Metric
- removed R9: 4.7k, Resistor_SMD:R_0805_2012Metric
- D1, D2: footprint Diode_SMD:D_0201_0603Metric -> Diode_SMD:D_0603_1608Metric
- J3: footprint Connector_FFC-FPC:TE_1-1734839-5_1x15-1MP_P0.5mm_Horizontal -> MyButtons:FPC-SMD_15P-P0.50_KH-FG0.5-H2.0-15P-SMT; moved to B.Cu
- J4: footprint Connector_FFC-FPC:TE_0-1734839-5_1x05-1MP_P0.5mm_Horizontal -> Connector_PinHeader_2.54mm:PinHeader_1x03_P2.54mm_Vertical
- moved C13 31.3 mm to (169.3, 83.2)
- moved U2 30.1 mm to (164.8, 107.2), turned to 90 degrees
- moved R5 29.5 mm to (158.1, 111.4)
- moved C8 29.1 mm to (167.5, 107.1), turned to -90 degrees
- moved C9 28.9 mm to (169.2, 107.1), turned to -90 degrees
- moved R6 28.5 mm to (160.2, 111.4), turned to 90 degrees
- moved U5 26.6 mm to (169.4, 86.2), turned to 90 degrees
- moved R2 24.6 mm to (168.6, 89.5)
- moved C5 23.7 mm to (149.1, 108.0)
- moved J2 23.6 mm to (152.1, 85.2)
- moved C15 23.6 mm to (149.1, 104.6)
- moved J4 20.6 mm to (151.8, 103.9), turned to 0 degrees
- moved SW1 18.5 mm to (167.6, 94.7), turned to 90 degrees
- moved R4 18.3 mm to (167.9, 103.1), turned to 0 degrees
- moved J1 18.1 mm to (148.2, 96.7), turned to 180 degrees
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Connections:
- C1 pad 2: VDD -> VDDSHUNTL
- C2 pad 2: VDD -> VDDSHUNTL
- C3 pad 2: VDD -> VDDSHUNTL
- C4 pad 2: VDD -> VDDSHUNTL
- J1 pad 1: Net-(J1-Pin_1) -> SWCLK
- J1 pad 2: Net-(J1-Pin_2) -> SWDIO
- J3 pad 12: TP_RST -> LCD_RST
- J3 pad 9: RST -> LCD_RST
- R2 pad 1: BATSHUNTH -> BATSHUNTL
- R4 pad 1: VDD -> VDDSHUNTL
- SW1 pad 1: BATSHUNTH -> BATSHUNTL
- U1 pad 1: VDD -> VDDSHUNTL
- U1 pad 17: VDD -> VDDSHUNTL
- U1 pad 21: USB_DM -> USB_D-
- U1 pad 22: USB_DP -> USB_D+
- U1 pad 30: TP_RST -> LCD_RST
- U1 pad 5: VDD -> VDDSHUNTL
- U6 pad 11: BATSHUNTH -> BATSHUNTL
- U6 pad 14: VDD -> VDDSHUNTL
- U8 pad 1: Net-(J5-D+) -> USB_D+
- U8 pad 3: Net-(J5-D-) -> USB_D-
- U8 pad 4: USB_DM -> Net-(J5-D-)
- U8 pad 6: USB_DP -> Net-(J5-D+)
Routing:
- net GND: track 0.00 -> 85.5 mm, vias 0 -> 36
- net BAT: track 0.00 -> 71.1 mm, vias 0 -> 3
- net CHARGE: track 0.00 -> 61.5 mm, vias 0 -> 2
- net I2C1_SDA: track 0.00 -> 46.2 mm, vias 0 -> 3
- net I2C1_SCL: track 0.00 -> 45.0 mm, vias 0 -> 2
- net VDDSHUNTL: track 0.00 -> 37.5 mm, vias 0 -> 3
- net LEDA: track 0.00 -> 31.5 mm, vias 0 -> 1
- net VDD: track 0.00 -> 29.6 mm, vias 0 -> 17
- net GYRO_INT2: track 0.00 -> 28.2 mm, vias 0 -> 4
- net SWCLK: track 0.00 -> 22.8 mm, vias 0 -> 1
- net SWDIO: track 0.00 -> 22.5 mm, vias 0 -> 1
- net LCD_RST: track 0.00 -> 22.5 mm, vias 0 -> 1
- net BATSHUNTL: track 0.00 -> 21.6 mm, vias 0 -> 2
- net USB_D-: track 0.00 -> 19.8 mm, vias 0 -> 2
- net USB_D+: track 0.00 -> 19.4 mm, vias 0 -> 2
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Other:
- board size 36 x 36 mm -> 40 x 40 mm
- board text added: "0"
- board text added: "5V"
- board text added: "HAOUT"
- board text added: "VDD"
- board text removed: "15"
- board text removed: "5"
- board text removed: "5v"
- board text removed: "BAT+"
